File: PCBs/Projects/MotorController/Main.sch (EAGLE design)
At the start: 129 parts, among them Q1 ZXMP10A17GQ, Q2 MMBT5551LT1G, Q3 BUK9240-100A.118, Q4 BUK9240-100A.118, U1 DRV8301, U11 LT4356-2, U2 ESDA6V1SC6Y, U3 ESDA6V1SC6Y, U4 ESDA6V1SC6Y, U5 TMP101, U6 ACS758LCB, U7 ESDA6V1SC6Y, U8 MTI85W100GC

Commit message: Starting work on Rev C, Rev B has been abandoned but not forgotten -Adding datasheets of some the the parts rec C will utilize -Added some power supply calculations -Added LT3045 and LT8631 parts in the IC library
Parts:
- removed C11, C9: 22n, SparkFun-Capacitors:CAP0805
- removed C16, C19: 0.1u, SparkFun-Capacitors:CAP0805
- removed C17: 2.2u, SparkFun-Capacitors:CAP1210
- removed C18: 4.7u, SparkFun-Capacitors:CAP1210
- removed C7, C8: 1u, SparkFun-Capacitors:CAP0805
- removed D5: PMEG10030ELPX, SparkFun-DiscreteSemi:PMEG10030ELPX
- removed R13: 16.2K, SparkFun-Resistors:RESISTOR0805-RES
- removed R14: 250k, SparkFun-Resistors:RESISTOR0805-RES
- removed R16: 100, SparkFun-Resistors:RESISTOR0805-RES
- removed R17: 51k, SparkFun-Resistors:RESISTOR0805-RES
- removed R18: 10k, SparkFun-Resistors:RESISTOR0805-RES
- removed SJ2: SOLDERJUMPERTRACE, SparkFun-Retired:SOLDERJUMPERTRACE
- removed U1: DRV8301, IC:DRV8301
- added FRAME8: FRAME-LEDGER, SparkFun-Aesthetics:FRAME-LEDGER
- C4: value 6.8N -> 0.1u
- C5: value 120P -> 0.1u
- C6: value 22n -> 0.1u
Connections:
- removed net 3.3V: C9.1, U1.VDD_SPI
- removed net IND_LOOP_IN: C16.2, D5.C, L1.1, U1.PH
- removed net N$10: C8.1, U1.AVDD
- removed net N$12: C6.1, U1.SS_TR
- removed net N$14: R17.1, R18.2, U1.VSENSE
- removed net N$15: C16.1, U1.BST_BK
- removed net N$17: C11.2, U1.CP2
- removed net N$18: C11.1, U1.CP1
- removed net N$21: C17.1, U1.GVDD
- removed net N$26: R16.1, U1.DTC
- removed net N$45: SJ2.2, U1.PWRGD
- removed net N$6: C5.1, R13.1, U1.COMP
- net !CS: no longer U1.!SCS
- net !FAULT: no longer U1.!FAULT
- net !OCTW: no longer U1.!OCTW
- net A: now also C6.2; no longer U1.SH_A
- net B: now also C5.2; no longer U1.SH_B
- net BUCK-EN: no longer U1.EN_BUCK
- net C: now also C4.2; no longer U1.SH_C
- net EN_GATE: no longer U1.EN_GATE
- net GH_A: no longer U1.GH_A
- net GH_B: no longer U1.GH_B
- net GH_C: no longer U1.GH_C
- net GL_A: no longer U1.GL_A
- net GL_B: no longer U1.GL_B
- net GL_C: no longer U1.GL_C
- net GND: no longer C17.2, C18.1, C19.2, C4.2, C5.2, C6.2, C7.2, C8.2, C9.2, D5.A, R14.1, R16.2, R18.1, U1.AGND, U1.GND(EXP_PAD), U1.SL_A, U1.SL_B, U1.SL_C, U1.SN1, U1.SN2, U1.SP1, U1.SP2
- net IND_LOOP_OUT: no longer L1.2, R17.2
- net INH_A: no longer U1.INH_A
- net INH_B: no longer U1.INH_B
- net INH_C: no longer U1.INH_C
- net INL_A: no longer U1.INL_A
- net INL_B: no longer U1.INL_B
- net INL_C: no longer U1.INL_C
- net MISO: no longer U1.SDO
- net MOSI: no longer U1.SDI
- net N$2: now also C6.1; no longer R14.2, U1.RT_CLK
- net N$24: no longer U1.BST_A
- net N$25: no longer U1.BST_C
- net N$3: no longer R13.2
- net N$30: no longer U1.BST_B
- net N$5: now also C5.1; no longer C7.1, U1.DVDD
- net PWRGD: no longer R15.1, SJ2.1
- net SCLK: no longer U1.SCLK
- net VCC: no longer C18.2, C19.1, U1.PVDD1, U1.PVDD2
Other:
- note removed: "1% max"
