File: PCBs/Projects/MotorController/Main.sch (EAGLE design)
At the start: 114 parts, among them Q1 ZXMP10A17GQ, Q2 MMBT5551LT1G, Q3 BUK9240-100A.118, Q4 BUK9240-100A.118, U11 LT4356-2, U2 ESDA6V1SC6Y, U3 ESDA6V1SC6Y, U4 ESDA6V1SC6Y, U5 TMP101, U6 ACS758LCB, U7 ESDA6V1SC6Y, U8 MTI85W100GC

Commit message: Gate driver circuitry added, many schematic updates -Some parts and datasheets also added
Parts:
- removed C21, C22: 47u, SparkFun-Capacitors:CAP1210
- removed FRAME8: FRAME-LEDGER, SparkFun-Aesthetics:FRAME-LEDGER
- removed L2: (no value), dp_devices.v6:FERRITE-1206
- removed SJ1: SOLDERJUMPERTRACE, SparkFun-Retired:SOLDERJUMPERTRACE
- removed SJ3: SOLDERJUMPERNO, SparkFun-Retired:SOLDERJUMPERNO
- added C11, C34, C8: 0.1u, SparkFun-Capacitors:CAP0805
- added C16, C17: 47u, SparkFun-Capacitors:CAP1210
- added C18, C19: 10u, SparkFun-Capacitors:CAP1210
- added C32: 4.7, SparkFun-Capacitors:CAP_POL1206
- added C33: 4.7u, SparkFun-Capacitors:CAP1210
- added C7: 2.2u, SparkFun-Capacitors:CAP1210
- added C9: 0.01u, SparkFun-Capacitors:CAP0805
- added D13, D5: GREEN, SparkFun-LED:LED-RED1206
- added Q5, Q7: NCV8440, SparkFun-DiscreteSemi:MOSFET-NCHANNELNCV8440
- added R13: 124k, SparkFun-Resistors:RESISTOR0805-RES
- added R14, R55: 10k, SparkFun-Resistors:RESISTOR0805-RES
- added R16: 25.5k, SparkFun-Resistors:RESISTOR0805-RES
- added R17: 1M, SparkFun-Resistors:RESISTOR0805-RES
- added R18: 57.6k, SparkFun-Resistors:RESISTOR0805-RES
- added R50, R53: 10, SparkFun-Resistors:RESISTOR0805-RES
- added R51: 0.5, SparkFun-Resistors:RESISTOR0805-RES
- added R52, R58: 47k, SparkFun-Resistors:RESISTOR0805-RES
- added R54: 140k, SparkFun-Resistors:RESISTOR0805-RES
- added R56: 2, SparkFun-Passives:RESISTOR1206
- added R57: 1k, SparkFun-Resistors:RESISTOR0805-RES
- added SJ2: SOLDERJUMPERNO, SparkFun-Retired:SOLDERJUMPERNO
- added U1: LT8631, IC:LT8631
- added U12, U13, U14: UCC27211A-Q1, IC:UCC27211A-Q1
- added U9: LT3045, IC:LT3045
- C10: value 0.1u -> 2.2u; device SparkFun-Capacitors:CAP0805 -> SparkFun-Capacitors:CAP1210
- C13: value 0.1u -> 200p
- C14: value 0.1u -> 5600p; device SparkFun-Capacitors:CAP0805 -> SparkFun-Capacitors:CAP1210
- C15: value 0.1u -> 47u; device SparkFun-Capacitors:CAP0805 -> SparkFun-Capacitors:CAP1210
- C20: value 47u -> DNP; device SparkFun-Capacitors:CAP1210 -> SparkFun-Capacitors:CAP0805
- C23: value 0.01u -> 0.1u
- C26, C27, C28, C29: value 10n -> 0.01u
- C4, C6: value 0.1u -> 4.7u; device SparkFun-Capacitors:CAP0805 -> SparkFun-Capacitors:CAP1210
- R11: value 274K -> 4.99k; device SparkFun-Resistors:RESISTOR1206 -> SparkFun-Resistors:RESISTOR0805-RES
- R12: value 4.99K -> 274k; device SparkFun-Resistors:RESISTOR1206 -> SparkFun-Resistors:RESISTOR0805-RES
- R15: value 47k -> 499
- R19: value 10 -> 2.7k
- R2: value 30k -> 47k; device SparkFun-Resistors:RESISTOR1206 -> SparkFun-Resistors:RESISTOR0805-RES
- R24, R25, R26: value 330 -> 1k
- R3: value 51 -> 100; device SparkFun-Resistors:RESISTOR1206 -> SparkFun-Resistors:RESISTOR0805-RES
- R5: device SparkFun-Resistors:RESISTOR1206 -> SparkFun-Resistors:RESISTOR0805-RES
- R6: value 133k -> 124k
Connections:
- net !IN-FAULT renamed !VIN-FAULT
- removed net BUCK-EN: SJ1.2
- removed net IND_LOOP_OUT: C20.1, C21.1, L2.2
- removed net PREJUMP_5V: C22.1, C23.1, L2.1, SJ3.1
- removed net PWRGD: MOD1.P_XRES
- new net 15V: C13.1, C15.1, C16.1, C17.1, C33.1, C4.1, C6.1, R17.2, R19.2, R52.2, R56.1, R57.2, U1.VOUT, U12.VDD, U13.VDD, U14.VDD
- new net 15V_PG: Q5.G, R52.1, U1.PG, U9.EN/UV
- new net 5V_PG: Q7.G, R58.1, U9.PG
- new net 5V_SET_CONNECTION: C32.+, R53.1, U9.SET
- new net ILIMIT_5V: R15.1, U9.ILIM
- new net N$10: L1.2, U1.IND
- new net N$12: C8.1, U1.BST
- new net N$14: C9.1, R13.1, R14.2, U1.EN/UV
- new net N$15: C10.1, U1.INTVCC
- new net N$17: R16.2, U1.RT
- new net N$18: C14.1, U1.TR/SS
- new net N$21: C13.2, C20.1, R17.1, R18.2, U1.FB
- new net N$26: C7.2, R51.2
- new net N$29: D5.C, Q5.D
- new net N$45: D13.A, R57.1
- new net N$6: C8.2, L1.1, U1.SW
- new net PG_FB: R54.2, R55.1, U9.PGFB
- net 5V: now also C19.1, R54.1, R58.2, U9.OUT, U9.OUTS; no longer R15.2, SJ3.2
- net A: now also C5.2, U12.HS; no longer C13.2, C6.2
- net B: now also C23.2, U13.HS; no longer C14.2, C5.2
- net C: now also C34.2, U14.HS; no longer C15.2, C4.2
- net FB: now also R11.2, R12.1; no longer R11.1, R12.2
- net GH_A: now also U12.HO
- net GH_B: now also U13.HO
- net GH_C: now also U14.HO
- net GL_A: now also U12.LO
- net GL_B: now also U13.LO
- net GL_C: now also U14.LO
- net GND: now also C11.2, C14.2, C15.2, C16.2, C17.2, C18.2, C19.2, C32.-, C33.2, C4.2, C6.2, C9.2, Q5.S, Q7.S, R11.1, R14.1, R15.2, R16.1, R18.1, R50.1, R51.1, R53.2, R55.2, U1.GND, U1.SYNC/MODE, U12.VSS, U13.VSS, U14.VSS, U9.GND; no longer C12.2, C21.2, C23.2, R12.1, R19.2
- net INH_A: now also U12.HI
- net INH_B: now also U13.HI
- net INH_C: now also U14.HI
- net INL_A: now also U12.LI
- net INL_B: now also U13.LI
- net INL_C: now also U14.LI
- net N$2: now also C5.1, U12.HB; no longer C6.1
- net N$24: now also C18.1, R56.2, U9.IN; no longer C13.1
- net N$25: now also C12.2, R50.2; no longer C15.1
- net N$3: now also C23.1, U13.HB; no longer C4.1
- net N$30: now also MOD1.P_XRES, SJ2.1; no longer C14.1
- net N$40: now also D5.A; no longer C22.2
- net N$46: now also D13.C, Q7.D; no longer SJ1.1, U11.EN
- net N$5: now also C34.1, U14.HB; no longer C5.1
- net VCC: now also C11.1, C7.1, R12.2, R13.2, U1.VIN; no longer C10.1, R11.2
Other:
- note added: "Gate Drivers"
- note added: "Kelvin Connections"
- note added: "Output limited to 70v and 250mA"
- note added: "Power Good LED 15v Supply"
- note added: "Power Good LED 5v Supply"
- note added: "Power Supplies"
- note added: "Power good when 5v rail is >4.5v"
- note added: "Tantalum"
- note added: "UVLO = ~16v"
- note removed: "74279221601"
- note removed: "Gate Driver and Buck Conv."
- note removed: "Gate Driver and Power Supply"
- note removed: "Output limited to 60v and 3A"

Commit message: Bulk of schematic work finished, beginning layout
Parts:
- removed MOD1: PSOC5LP-DEVBRDCY8CKIT-059, modules:PSOC5LP-DEVBRDCY8CKIT-059
- removed SJ2: SOLDERJUMPERNO, SparkFun-Retired:SOLDERJUMPERNO
- added C21, C22: 0.1u, SparkFun-Capacitors:CAP0805
- added D14, D15, D16: 1SMA15AT3G, SparkFun-DiscreteSemi:TVSSMA
- added FD4, FD5, FD6: FIDUCIAL1X2, SparkFun-Aesthetics:FIDUCIAL1X2
- added MOD2: PSOC5LP-DEVBRDCY8CKIT-059, modules:PSOC5LP-DEVBRDCY8CKIT-059
- added R59, R60, R61, R62: 100, SparkFun-Resistors:RESISTOR0805-RES
- added SW1: DIP-SWTCH-16POSCD16RM0SBR, SparkFun-Electromechanical:DIP-SWTCH-16POSCD16RM0SBR
- D10, D11, D12, D7, D8, D9: value MBRF1090 -> MBRF10H100
- R4: device SparkFun-Passives:RESISTOR1206 -> SparkFun-Resistors:RESISTOR0805-RES
Connections:
- removed net !CS: MOD1.P1_2
- removed net !FAULT: MOD1.P1_6
- removed net !OCTW: MOD1.P1_7
- removed net EN_GATE: MOD1.P12_2
- removed net MISO: MOD1.P1_4
- removed net MOSI: MOD1.P1_3
- removed net SCLK: MOD1.P1_5
- new net 15V1: D15.C
- new net 15V2: D16.C
- new net GND1: D15.A
- new net GND2: D16.A
- new net MODESET1: SW1.1
- new net MODESET2: SW1.2
- new net MODESET3: R61.1, SW1.4
- new net MODESET4: R62.1, SW1.8
- new net N$53: MOD2.P3_1, R60.2
- new net N$54: MOD2.P3_0, R59.2
- new net N$55: MOD2.P3_4, R62.2
- net !VIN-FAULT: no longer MOD1.P1_1
- net 15V: now also D14.C
- net 5V: now also C21.1, C22.1; no longer MOD1.VDD, MOD1.VDDIO
- net GND: now also C21.2, C22.2, D14.A, SW1.C; no longer MOD1.GND
- net INH_A: no longer MOD1.P12_3
- net INH_B: no longer MOD1.P12_5
- net INH_C: no longer MOD1.P12_7
- net INL_A: no longer MOD1.P12_4
- net INL_B: no longer MOD1.P12_6
- net INL_C: no longer MOD1.P2_7
- net ISENSE: no longer MOD1.P3_1
- net N$16: no longer MOD1.P2_3
- net N$30: now also MOD2.P3_3, R61.2; no longer MOD1.P_XRES, SJ2.1
- net N$32: no longer MOD1.P2_6
- net N$33: no longer MOD1.P2_5
- net N$34: no longer MOD1.P2_4
- net N$39: no longer MOD1.P3_4
- net N$41: no longer MOD1.P2_2
- net N$42: no longer MOD1.P0_6
- net N$43: no longer MOD1.P15_3
- net N$44: no longer MOD1.P15_5
- net N$47: no longer MOD1.P15_1
- net N$48: no longer MOD1.P15_2
- net N$49: no longer MOD1.P0_7
- net N$8: no longer MOD1.P15_0
- net SCL: no longer MOD1.P3_6
- net SDA: no longer MOD1.P3_7
- net T_ALERT: no longer MOD1.P0_5
- net VSENSE: no longer MOD1.P3_0
Other:
- note added: "Bottom Layer"
- note added: "DNP"
- note added: "Phase Combination Selector"
- moved on the sheet: C25, D6, R20, R21, R22, R23, R24, R25, R26, R27, R28, R29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

Commit message: Added test points to schematic -Restarted board
Parts:
- removed U14: UCC27211A-Q1, IC:UCC27211A-Q1
- added C35: 0.01u, SparkFun-Capacitors:CAP0805
- added F1, F2: B59607A120A62, SparkFun-PowerIC:PTC1210
- added TP1, TP10, TP11, TP12, TP13, TP14, TP15, TP16, TP17, TP2, TP3, TP4, TP5, TP6, TP7, TP8, TP9: TEST-POINTRCT-0C, SparkFun-Passives:TEST-POINTRCT-0C
- added U10: UCC27211A-Q1, IC:UCC27211A-Q1
- C10: value 2.2u -> 5600p
- C12: value 4.7u -> 4.7; device SparkFun-Capacitors:CAP1210 -> SparkFun-Capacitors:CAP_POL1206
- C14: value 5600p -> DNP; device SparkFun-Capacitors:CAP1210 -> SparkFun-Capacitors:CAP0805
- C16: value 47u -> 10u
- C18: value 10u -> 47u
- C19: value 10u -> 0.1u; device SparkFun-Capacitors:CAP1210 -> SparkFun-Capacitors:CAP0805
- C20: value DNP -> 0.1u
- C23, C24, C25, C8: value 0.1u -> 0.01u
- C27, C31: value 0.01u -> 0.1u
- C28, C29: value 0.01u -> 4.7u; device SparkFun-Capacitors:CAP0805 -> SparkFun-Capacitors:CAP1210
- C30: value 0.1u -> 4.7u; device SparkFun-Capacitors:CAP0805 -> SparkFun-Capacitors:CAP1210
- C32: value 4.7 -> 0.1u; device SparkFun-Capacitors:CAP_POL1206 -> SparkFun-Capacitors:CAP0805
- C33, C6: value 4.7u -> 0.1u; device SparkFun-Capacitors:CAP1210 -> SparkFun-Capacitors:CAP0805
- C5: value 0.1u -> 2.2u; device SparkFun-Capacitors:CAP0805 -> SparkFun-Capacitors:CAP1210
- C7: value 2.2u -> 10u
- C9: value 0.01u -> 2.2u; device SparkFun-Capacitors:CAP0805 -> SparkFun-Capacitors:CAP1210
- D10, D8, D9: value MBRF10H100 -> 1SMA15AT3G; device SparkFun-DiscreteSemi:DIODE-SCHOTTKY-MBRF1090_V -> SparkFun-DiscreteSemi:TVSSMA
- D13: value GREEN -> MBRF10H100; device SparkFun-LED:LED-RED1206 -> SparkFun-DiscreteSemi:DIODE-SCHOTTKY-MBRF1090_V
- D14, D15, D16: value 1SMA15AT3G -> MBRF10H100; device SparkFun-DiscreteSemi:TVSSMA -> SparkFun-DiscreteSemi:DIODE-SCHOTTKY-MBRF1090_V
- D6: value CLV1A-FKB -> GREEN; device SparkFun-LED:0.13_RGB_LEDCLV1A-FKB -> SparkFun-LED:LED-RED1206
- D7: value MBRF10H100 -> CLV1A-FKB; device SparkFun-DiscreteSemi:DIODE-SCHOTTKY-MBRF1090_V -> SparkFun-LED:0.13_RGB_LEDCLV1A-FKB
- R11: value 4.99k -> 274k
- R12: value 274k -> 4.99k
- R13: value 124k -> 10
- R14: value 10k -> 0.5
- R15: value 499 -> 2; device SparkFun-Resistors:RESISTOR0805-RES -> SparkFun-Passives:RESISTOR1206
- R16: value 25.5k -> 124k
- R17: value 1M -> 10k
- R18: value 57.6k -> 47k
- R19: value 2.7k -> 25.5k
- R20: value 100 -> 499
- R21: value 100 -> 47k
- R22: value 100 -> 1M
- R23: value 100 -> 57.6k
- R24, R57: value 1k -> 10
- R25: value 1k -> 140k
- R26: value 1k -> 10k
- R27: value 100 -> 2.7k
- R28: value 100 -> 1k
- R33: value 510k -> 4.7k
- R34, R35: value 1k -> 100
- R36, R37: value 4.7k -> 100
- R38, R39, R40: value 10k -> 100
- R41: value 100k -> 100; device SparkFun-Resistors:RESISTOR1206 -> SparkFun-Resistors:RESISTOR0805-RES
- R42: value 5.1k -> 1k; device SparkFun-Resistors:RESISTOR1206 -> SparkFun-Resistors:RESISTOR0805-RES
- R43, R44: value 10 -> 1k
- R45, R47: value 10 -> 100
- R46: value 10 -> 4.7k
- R48: value 10 -> 100k; device SparkFun-Resistors:RESISTOR0805-RES -> SparkFun-Resistors:RESISTOR1206
- R49: value 1M -> 5.1k
- R50: value 10 -> 10k
- R51: value 0.5 -> 10k
- R52: value 47k -> 10k
- R53: value 10 -> 510k
- R54: value 140k -> 1k
- R55: value 10k -> 1k
- R56: value 2 -> 10; device SparkFun-Passives:RESISTOR1206 -> SparkFun-Resistors:RESISTOR0805-RES
- R58: value 47k -> 10
- R59, R60, R61: value 100 -> 10
- R62: value 100 -> 1M; device SparkFun-Resistors:RESISTOR0805-RES -> SparkFun-Resistors:RESISTOR1206
- R8: value 0.016 -> 0.2
- U1: value LT8631 -> LT4356-2; device IC:LT8631 -> IC:LT4356-2
- U11: value LT4356-2 -> UCC27211A-Q1; device IC:LT4356-2 -> IC:UCC27211A-Q1
- U13: value UCC27211A-Q1 -> MTI85W100GC; device IC:UCC27211A-Q1 -> IC:MTI85W100GC
- U2: value ESDA6V1SC6Y -> LT8631; device IC:ESDA6V1SC6Y -> IC:LT8631
- U3: value ESDA6V1SC6Y -> LT3045; device IC:ESDA6V1SC6Y -> IC:LT3045
- U4: value ESDA6V1SC6Y -> TMP101; device IC:ESDA6V1SC6Y -> SparkFun-DigitalIC:TMP101
- U5: value TMP101 -> ACS758LCB; device SparkFun-DigitalIC:TMP101 -> IC:ACS758LCB
- U6: value ACS758LCB -> ESDA6V1SC6Y; device IC:ACS758LCB -> IC:ESDA6V1SC6Y
- U8: value MTI85W100GC -> ESDA6V1SC6Y; device IC:MTI85W100GC -> IC:ESDA6V1SC6Y
- U9: value LT3045 -> ESDA6V1SC6Y; device IC:LT3045 -> IC:ESDA6V1SC6Y
- renumbered MOD2 to MOD1, Q7 to Q6
Connections:
- removed net N$41 (its old number): R22.2
- removed net N$49 (its old number): R21.2
- new net N$47: R39.2
- new net N$48: R40.2
- new net N$56: F1.2, J4.1
- new net N$57: C34.1, F2.1, J5.5
- net !VIN-FAULT: now also U1.!FAULT; no longer U11.!FAULT
- net 15V: now also C18.1, C28.1, C29.1, C30.1, D10.C, R15.1, R21.2, R22.2, R27.2, R28.2, TP3.1, U10.VDD, U11.VDD, U2.VOUT; no longer C16.1, C33.1, C4.1, C6.1, D14.C, R17.2, R19.2, R52.2, R56.1, R57.2, U1.VOUT, U13.VDD, U14.VDD
- net 15V1: now also D9.C; no longer D15.C
- net 15V2: now also D8.C; no longer D16.C
- net 15V_PG: now also R21.1, U2.PG, U3.EN/UV; no longer R52.1, U1.PG, U9.EN/UV
- net 5V: now also C16.1, C20.1, C23.1, D7.ANODE, F1.1, F2.2, R18.2, R25.1, R33.1, R46.1, R50.1, R51.1, R52.1, TP2.1, U3.OUT, U3.OUTS, U4.V+, U5.VCC, U9.IO1; no longer C22.1, C28.1, C30.1, D6.ANODE, J4.1, J5.5, R34.1, R36.1, R37.1, R38.1, R39.1, R40.1, R58.2, U5.V+, U6.VCC, U7.IO1, U9.OUT, U9.OUTS
- net 5V_PG: now also R18.1, U3.PG; no longer R58.1, U9.PG
- net 5V_SET_CONNECTION: now also C12.+, R24.1, U3.SET; no longer C32.+, R53.1, U9.SET
- net A: now also C31.2, D11.A, D12.C, U10.HS, U13.L1, U13.S1; no longer C5.2, D7.A, D8.C, U12.HS, U8.L1, U8.S1
- net B: now also C32.2, D13.A, D14.C, U11.HS, U13.L2, U13.S3; no longer C23.2, D10.C, D9.A, U13.HS, U8.L2, U8.S3
- net C: now also C33.2, D15.A, D16.C, U12.HS, U13.L3, U13.S5; no longer C34.2, D11.A, D12.C, U14.HS, U8.L3, U8.S5
- net DISABLE: now also R45.1, U6.IO4; no longer R23.1, U2.IO4
- net DISP_OUT: now also R31.1, U8.IO3; no longer R22.1, U4.IO3
- net FB: now also R11.1, R12.2, U1.FB; no longer R11.2, R12.1, U11.FB
- net GATEDRV: now also U1.GATE; no longer U11.GATE
- net GH_A: now also R56.2, TP17.1, U10.HO; no longer R43.2, U12.HO
- net GH_B: now also R58.2, TP15.1, U11.HO; no longer R45.2, U13.HO
- net GH_C: now also R60.2, TP13.1, U12.HO; no longer R47.2, U14.HO
- net GL_A: now also R57.2, TP16.1, U10.LO; no longer R44.2, U12.LO
- net GL_B: now also R59.2, TP14.1, U11.LO; no longer R46.2, U13.LO
- net GL_C: now also R61.2, TP12.1, U12.LO; no longer R48.2, U14.LO
- net GND: now also C12.-, C27.2, C28.2, C34.2, C35.2, C7.2, C8.2, D16.A, R12.1, R13.1, R17.1, R19.1, R20.2, R23.1, R24.2, R26.2, R62.1, U10.VSS, U11.VSS, U13.L-, U13.S2, U13.S4, U13.S6, U2.SYNC/MODE, U4.ADD0, U8.GND; no longer C11.2, C24.2, C31.2, C32.-, C33.2, C4.2, D8.A, R11.1, R15.2, R16.1, R18.1, R33.2, R35.2, R42.1, R50.1, R51.1, U1.SYNC/MODE, U11.GND, U13.VSS, U14.VSS, U5.ADD0, U8.L-, U8.S2, U8.S4, U8.S6
- net GND1: now also D9.A; no longer D15.A
- net GND2: now also D8.A; no longer D16.A
- net GPIO_TBD: now also R41.1, U8.IO4; no longer R20.1, U4.IO4
- net H1: now also C23.2, R38.1, R50.2, TP6.1, U9.IO2; no longer C26.2, R28.1, R38.2, U7.IO2
- net H2: now also C24.2, R39.1, R51.2, TP7.1, U9.IO3; no longer C27.2, R29.1, R39.2, U7.IO3
- net H3: now also C26.2, R40.1, R52.2, TP8.1, U9.IO4; no longer C28.2, R30.1, R40.2, U7.IO4
- net ILIMIT_5V: now also R20.1, U3.ILIM; no longer R15.1, U9.ILIM
- net INH_A: now also U10.HI; no longer U12.HI
- net INH_B: now also U11.HI; no longer U13.HI
- net INH_C: now also U12.HI; no longer U14.HI
- net INL_A: now also U10.LI; no longer U12.LI
- net INL_B: now also U11.LI; no longer U13.LI
- net INL_C: now also U12.LI; no longer U14.LI
- net ISENSE: now also C25.1, TP10.1, U5.VIOUT, U7.IO3; no longer C29.1, U3.IO3, U6.VIOUT
- net MODESET3: now also R36.1; no longer R61.1
- net MODESET4: now also R37.1; no longer R62.1
- net MONITOR_RX: now also R30.1, U8.IO2; no longer R32.1, U4.IO2
- net MONITOR_TX: now also R29.1, U8.IO1; no longer R31.1, U4.IO1
- net N$1: now also U1.TMR; no longer U11.TMR
- net N$10: now also U2.IND; no longer U1.IND
- net N$12: now also C11.1, U2.BST; no longer C8.1, U1.BST
- net N$13: now also U1.IN+; no longer U11.IN+
- net N$14: now also C8.1, R16.1, R17.2, U2.EN/UV; no longer C9.1, R13.1, R14.2, U1.EN/UV
- net N$15: now also C9.1, U2.INTVCC; no longer C10.1, U1.INTVCC
- net N$16: now also R45.2; no longer R23.2
- net N$17: now also R19.2, U2.RT; no longer R16.2, U1.RT
- net N$18: now also C10.1, U2.TR/SS; no longer C14.1, U1.TR/SS
- net N$2: now also C31.1, U10.HB; no longer C5.1, U12.HB
- net N$21: now also C14.1, R22.1, R23.2, U2.FB; no longer C20.1, R17.1, R18.2, U1.FB
- net N$24: now also C7.1, R15.2, U3.IN; no longer C18.1, R56.2, U9.IN
- net N$25: now also C4.2, R13.2; no longer C12.2, R50.2
- net N$26: now also C5.2, R14.2; no longer C7.2, R51.2
- net N$27: now also R58.1, U13.G3; no longer R45.1, U8.G3
- net N$28: now also R56.1, U13.G1; no longer R43.1, U8.G1
- net N$3: now also C32.1, U11.HB; no longer C23.1, U13.HB
- net N$30: now also R36.2; no longer R61.2
- net N$31: now also C35.1, R62.2; no longer C31.1, R49.2
- net N$32: now also R44.1; no longer R26.1
- net N$33: now also R43.1; no longer R25.1
- net N$34: now also R42.1; no longer R24.1
- net N$35: now also D7.RED, R44.2; no longer D6.RED, R26.2
- net N$36: now also D7.GREEN, R43.2; no longer D6.GREEN, R25.2
- net N$37: now also D7.BLUE, R42.2; no longer D6.BLUE, R24.2
- net N$38: now also R57.1, U13.G2; no longer R44.1, U8.G2
- net N$39: now also C22.1, R47.2, TP11.1; no longer C25.1, R27.2
- net N$40: now also R27.1; no longer R19.1
- net N$42: now also R41.2; no longer R20.2
- net N$45: now also D6.A, R28.1; no longer D13.A, R57.1
- net N$46: now also D6.C; no longer D13.C
- net N$5: now also C33.1, U12.HB; no longer C34.1, U14.HB
- net N$50: now also R59.1, U13.G4; no longer R46.1, U8.G4
- net N$51: now also R60.1, U13.G5; no longer R47.1, U8.G5
- net N$52: now also R61.1, U13.G6; no longer R48.1, U8.G6
- net N$53: now also R35.2; no longer R60.2
- net N$54: now also R34.2; no longer R59.2
- net N$55: now also R37.2; no longer R62.2
- net N$6: now also C11.2, U2.SW; no longer C8.2, U1.SW
- net N$8: now also R38.2; no longer R28.2
- net PG_FB: now also R25.2, R26.1, U3.PGFB; no longer R54.2, R55.1, U9.PGFB
- net POST-SENSE: now also U1.SNS; no longer U11.SNS
- net PRE-SENSE: now also U1.!SHDN, U1.VCC; no longer U11.!SHDN, U11.VCC
- net REVERSE: now also R32.1, U6.IO3; no longer R21.1, U2.IO3
- net SCL: now also R33.2, TP4.1, U4.SCL; no longer R36.2, U5.SCL
- net SDA: now also R46.2, TP5.1, U4.SDA; no longer R37.2, U5.SDA
- net THROTTLE_1: now also R54.2, U6.IO1; no longer R34.2, U2.IO1
- net THROTTLE_2: now also R47.1, R53.1, U6.IO2; no longer R27.1, R33.1, U2.IO2
- net THROTTLE_3: now also R55.1; no longer R35.1
- net T_ALERT: now also U4.ALERT; no longer U5.ALERT
- net UNDERVOLTAGE: now also U1.AOUT; no longer U11.AOUT
- net VCC: now also C4.1, C5.1, C6.1, R11.2, R16.2, R48.2, TP1.1, U1.OUT, U2.VIN; no longer C11.1, C12.1, C7.1, R12.2, R13.2, R41.2, U1.VIN, U11.OUT
- net VIN: now also U5.IP+; no longer U6.IP+
- net VSENSE: now also R48.1, R49.2, U7.IO1; no longer R41.1, R42.2, U3.IO1
- net V_BATT: now also D13.C, D15.C, U13.L+, U5.IP-; no longer D7.C, D9.C, U6.IP-, U8.L+
Other:
- note added: "100mA PTC fuse"
