File: PCBs/Projects/MotorController/Main.sch (EAGLE design)
At the start: 174 parts, among them Q1 ZXMP10A17GQ, Q2 MMBT5551LT1G, Q3 BUK9240-100A.118, Q4 BUK9240-100A.118, Q5 NCV8440, Q6 NCV8440, SW1 DIP-SWTCH-16POSCD16RM0SBR, U1 LT4356-2, U10 UCC27211A-Q1, U11 UCC27211A-Q1, U12 UCC27211A-Q1, U13 MTI85W100GC, U2 LT8631, U3 LT3045, U4 TMP101, U5 ACS758LCB, U6 ESDA6V1SC6Y, U7 ESDA6V1SC6Y, U8 ESDA6V1SC6Y, U9 ESDA6V1SC6Y

Commit message: Most Layout complete
Connections:
- net DISP_OUT: now also U8.IO4; no longer U8.IO3
- net GPIO_TBD: now also U8.IO3; no longer U8.IO4
- net MONITOR_RX: now also U8.IO1; no longer U8.IO2
- net MONITOR_TX: now also U8.IO2; no longer U8.IO1
- net N$35: now also D7.BLUE; no longer D7.RED
- net N$37: now also D7.RED; no longer D7.BLUE
Changed lines of the file:
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@@
 <net name="MONITOR_TX" class="0">
 <segment>
-<pinref part="U8" gate="G$1" pin="IO1"/>
-<wire x1="373.38" y1="213.36" x2="388.62" y2="213.36" width="0.4064" layer="91"/>
+<pinref part="U8" gate="G$1" pin="IO2"/>
+<wire x1="373.38" y1="208.28" x2="388.62" y2="213.36" width="0.4064" layer="91"/>
 <label x="374.65" y="214.63" size="1.778" layer="95"/>
 </segment>
@@
 <net name="MONITOR_RX" class="0">
 <segment>
-<pinref part="U8" gate="G$1" pin="IO2"/>
-<wire x1="373.38" y1="208.28" x2="388.62" y2="208.28" width="0.4064" layer="91"/>
+<pinref part="U8" gate="G$1" pin="IO1"/>
+<wire x1="373.38" y1="213.36" x2="388.62" y2="208.28" width="0.4064" layer="91"/>
 <label x="374.65" y="209.55" size="1.778" layer="95"/>
 </segment>
@@
 </segment>
 <segment>
-<pinref part="U8" gate="G$1" pin="IO3"/>
-<wire x1="373.38" y1="203.2" x2="388.62" y2="203.2" width="0.4064" layer="91"/>
+<pinref part="U8" gate="G$1" pin="IO4"/>
+<wire x1="373.38" y1="198.12" x2="388.62" y2="203.2" width="0.4064" layer="91"/>
 <label x="375.92" y="203.2" size="1.778" layer="95"/>
 </segment>
@@
 </segment>
 <segment>
-<pinref part="U8" gate="G$1" pin="IO4"/>
-<wire x1="373.38" y1="198.12" x2="388.62" y2="198.12" width="0.4064" layer="91"/>
+<pinref part="U8" gate="G$1" pin="IO3"/>
+<wire x1="373.38" y1="203.2" x2="388.62" y2="198.12" width="0.4064" layer="91"/>
 <label x="375.92" y="198.12" size="1.778" layer="95"/>
 </segment>
@@
 <segment>
 <pinref part="R42" gate="G$1" pin="2"/>
-<wire x1="30.48" y1="147.32" x2="35.56" y2="147.32" width="0.4064" layer="91"/>
-<pinref part="D7" gate="G$1" pin="BLUE"/>
+<wire x1="30.48" y1="137.16" x2="35.56" y2="147.32" width="0.4064" layer="91"/>
+<pinref part="D7" gate="G$1" pin="RED"/>
 </segment>
 </net>
@@
 <segment>
 <pinref part="R44" gate="G$1" pin="2"/>
-<wire x1="35.56" y1="137.16" x2="30.48" y2="137.16" width="0.4064" layer="91"/>
-<pinref part="D7" gate="G$1" pin="RED"/>
+<wire x1="35.56" y1="137.16" x2="30.48" y2="147.32" width="0.4064" layer="91"/>
+<pinref part="D7" gate="G$1" pin="BLUE"/>
 </segment>
 </net>
