File: PCBs/Projects/MotorController/Main.brd (EAGLE design)
At the start: 172.7 x 99.1 mm, 114 parts, among them Q1 ZXMP10A17GQ, Q2 MMBT5551LT1G, Q3 BUK9240-100A.118, Q4 BUK9240-100A.118, U11 LT4356-2, U2 ESDA6V1SC6Y, U3 ESDA6V1SC6Y, U4 ESDA6V1SC6Y, U5 TMP101, U6 ACS758LCB, U7 ESDA6V1SC6Y, U8 MTI85W100GC

Commit message: Gate driver circuitry added, many schematic updates -Some parts and datasheets also added
Parts:
- removed C21, C22: 47u, SparkFun-Capacitors:1210
- removed FRAME8: FRAME-LEDGER, SparkFun-Aesthetics:CREATIVE_COMMONS
- removed L2: (no value), dp_devices.v6:FB1206
- removed SJ1: SOLDERJUMPERTRACE, SparkFun-Retired:SJ_2S-TRACE
- removed SJ3: SOLDERJUMPERNO, SparkFun-Retired:SJ_2S-NO
- added C11, C34, C8: 0.1u, SparkFun-Capacitors:0805
- added C16, C17: 47u, SparkFun-Capacitors:1210
- added C18, C19: 10u, SparkFun-Capacitors:1210
- added C32: 4.7, SparkFun-Capacitors:EIA3216
- added C33: 4.7u, SparkFun-Capacitors:1210
- added C7: 2.2u, SparkFun-Capacitors:1210
- added C9: 0.01u, SparkFun-Capacitors:0805
- added D13, D5: GREEN, SparkFun-LED:LED-1206
- added Q5, Q7: NCV8440, SparkFun-DiscreteSemi:SOT223
- added R13: 124k, SparkFun-Resistors:0805
- added R14, R55: 10k, SparkFun-Resistors:0805
- added R16: 25.5k, SparkFun-Resistors:0805
- added R17: 1M, SparkFun-Resistors:0805
- added R18: 57.6k, SparkFun-Resistors:0805
- added R50, R53: 10, SparkFun-Resistors:0805
- added R51: 0.5, SparkFun-Resistors:0805
- added R52, R58: 47k, SparkFun-Resistors:0805
- added R54: 140k, SparkFun-Resistors:0805
- added R56: 2, SparkFun-Passives:1206
- added R57: 1k, SparkFun-Resistors:0805
- added SJ2: SOLDERJUMPERNO, SparkFun-Retired:SJ_2S-NO
- added U1: LT8631, IC:TSSOP-20-FE
- added U12, U13, U14: UCC27211A-Q1, IC:SOIC-8-EP
- added U9: LT3045, IC:MSOP-12-EP
- C10: value 0.1u -> 2.2u; device SparkFun-Capacitors:0805 -> SparkFun-Capacitors:1210
- C13: value 0.1u -> 200p
- C14: value 0.1u -> 5600p; device SparkFun-Capacitors:0805 -> SparkFun-Capacitors:1210
- C15: value 0.1u -> 47u; device SparkFun-Capacitors:0805 -> SparkFun-Capacitors:1210
- C20: value 47u -> DNP; device SparkFun-Capacitors:1210 -> SparkFun-Capacitors:0805
- C23: value 0.01u -> 0.1u
- C26, C27, C28, C29: value 10n -> 0.01u
- C4, C6: value 0.1u -> 4.7u; device SparkFun-Capacitors:0805 -> SparkFun-Capacitors:1210
- R11: value 274K -> 4.99k; device SparkFun-Resistors:1206 -> SparkFun-Resistors:0805
- R12: value 4.99K -> 274k; device SparkFun-Resistors:1206 -> SparkFun-Resistors:0805
- R15: value 47k -> 499
- R19: value 10 -> 2.7k
- R2: value 30k -> 47k; device SparkFun-Resistors:1206 -> SparkFun-Resistors:0805
- R24, R25, R26: value 330 -> 1k
- R3: value 51 -> 100; device SparkFun-Resistors:1206 -> SparkFun-Resistors:0805
- R5: device SparkFun-Resistors:1206 -> SparkFun-Resistors:0805
- R6: value 133k -> 124k
- moved R5 300.3 mm to (-110.5, -160.7)
- moved R3 269.4 mm to (-87.0, -133.3), turned to 0 degrees
- moved R19 242.7 mm to (-104.1, -133.3), turned to 0 degrees
- moved C23 222.6 mm to (-83.8, -120.7), turned to 0 degrees
- moved R2 219.0 mm to (-83.8, -61.6)
- moved R12 193.3 mm to (-80.6, -61.6)
- moved R11 192.8 mm to (-77.5, -61.6), turned to 0 degrees
- moved C20 172.4 mm to (-74.3, -61.6), turned to 0 degrees
- moved C14 131.4 mm to (-50.8, -33.0)
- moved C15 129.9 mm to (-50.8, -36.2)
- moved C6 127.4 mm to (-80.0, -120.7)
- moved C13 124.5 mm to (-42.5, -29.2)
- moved C4 123.1 mm to (-80.0, -108.0)
- moved C5 122.1 mm to (-83.8, -108.0)
- moved C10 110.6 mm to (-25.4, -29.8), turned to 0 degrees
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Connections:
- net !IN-FAULT renamed !VIN-FAULT
- removed net BUCK-EN: SJ1.2
- removed net IND_LOOP_OUT: C20.1, C21.1, L2.2
- removed net PREJUMP_5V: C22.1, C23.1, L2.1, SJ3.1
- removed net PWRGD: MOD1.24
- new net 15V: C13.1, C15.1, C16.1, C17.1, C33.1, C4.1, C6.1, R17.2, R19.2, R52.2, R56.1, R57.2, U1.12, U12.1, U13.1, U14.1
- new net 15V_PG: Q5.1, R52.1, U1.5, U9.4
- new net 5V_PG: Q7.1, R58.1, U9.5
- new net 5V_SET_CONNECTION: C32.A, R53.1, U9.8
- new net ILIMIT_5V: R15.1, U9.6
- new net N$10: L1.P$2, U1.14
- new net N$12: C8.1, U1.18
- new net N$14: C9.1, R13.1, R14.2, U1.3
- new net N$15: C10.1, U1.16
- new net N$17: R16.2, U1.8
- new net N$18: C14.1, U1.10
- new net N$21: C13.2, C20.1, R17.1, R18.2, U1.11
- new net N$26: C7.2, R51.2
- new net N$29: D5.C, Q5.2, Q5.4
- new net N$45: D13.A, R57.1
- new net N$6: C8.2, L1.P$1, U1.20
- new net PG_FB: R54.2, R55.1, U9.7
- net 5V: now also C19.1, R54.1, R58.2, U9.10, U9.11, U9.12; no longer R15.2, SJ3.2
- net A: now also C5.2, U12.4; no longer C13.2, C6.2
- net B: now also C23.2, U13.4; no longer C14.2, C5.2
- net C: now also C34.2, U14.4; no longer C15.2, C4.2
- net FB: now also R11.2, R12.1; no longer R11.1, R12.2
- net GH_A: now also U12.3
- net GH_B: now also U13.3
- net GH_C: now also U14.3
- net GL_A: now also U12.8
- net GL_B: now also U13.8
- net GL_C: now also U14.8
- net GND: now also C11.2, C14.2, C15.2, C16.2, C17.2, C18.2, C19.2, C32.C, C33.2, C4.2, C6.2, C9.2, Q5.3, Q7.3, R11.1, R14.1, R15.2, R16.1, R18.1, R50.1, R51.1, R53.2, R55.2, U1.13, U1.15, U1.6, U1.7, U1.9, U1.EXP, U12.7, U12.EP1, U12.EP2, U12.EP3, U12.EP4, U12.EP5, U12.EP6, U12.EXP, U13.7, U13.EP1, U13.EP2, U13.EP3, U13.EP4, U13.EP5, U13.EP6, U13.EXP, U14.7, U14.EP1, U14.EP2, U14.EP3, U14.EP4, U14.EP5, U14.EP6, U14.EXP, U9.9, U9.EXP; no longer C12.2, C21.2, C23.2, R12.1, R19.2
- net INH_A: now also U12.5
- net INH_B: now also U13.5
- net INH_C: now also U14.5
- net INL_A: now also U12.6
- net INL_B: now also U13.6
- net INL_C: now also U14.6
- net N$2: now also C5.1, U12.2; no longer C6.1
- net N$24: now also C18.1, R56.2, U9.1, U9.2, U9.3; no longer C13.1
- net N$25: now also C12.2, R50.2; no longer C15.1
- net N$3: now also C23.1, U13.2; no longer C4.1
- net N$30: now also MOD1.24, SJ2.1; no longer C14.1
- net N$40: now also D5.A; no longer C22.2
- net N$46: now also D13.C, Q7.2, Q7.4; no longer SJ1.1, U11.11
- net N$5: now also C34.1, U14.2; no longer C5.1
- net VCC: now also C11.1, C7.1, R12.2, R13.2, U1.1; no longer C10.1, R11.2
Routing:
- net BUCK-EN: track 37.3 -> 0.00 mm, vias 2 -> 0
- net 5V: track 529.1 -> 521.5 mm
- net N$25: track 5.48 -> 0.00 mm
- net FB: track 11.1 -> 6.03 mm
- net N$46: track 2.61 -> 0.00 mm
- net UNDERVOLTAGE: track 17.8 -> 15.4 mm
- net N$30: track 1.85 -> 0.00 mm
- net N$7: track 5.45 -> 3.80 mm
- net N$24: track 1.61 -> 0.00 mm
- net N$40: track 1.56 -> 0.00 mm
- net B: track 22.0 -> 20.6 mm
- net A: track 31.2 -> 30.1 mm
- net C: track 26.4 -> 25.2 mm
- net N$20: track 44.3 -> 43.2 mm
- net PREJUMP_5V: track 0.90 -> 0.00 mm
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
Commit message: Bulk of schematic work finished, beginning layout
Parts:
- removed MOD1: PSOC5LP-DEVBRDCY8CKIT-059, modules:CYKIT059
- removed SJ2: SOLDERJUMPERNO, SparkFun-Retired:SJ_2S-NO
- added C21, C22: 0.1u, SparkFun-Capacitors:0805
- added D14, D15, D16: 1SMA15AT3G, SparkFun-DiscreteSemi:SMA-DIODE
- added FD4, FD5, FD6: FIDUCIAL1X2, SparkFun-Aesthetics:FIDUCIAL-1X2
- added MOD2: PSOC5LP-DEVBRDCY8CKIT-059, modules:CYKIT059
- added R59, R60, R61, R62: 100, SparkFun-Resistors:0805
- added SW1: DIP-SWTCH-16POSCD16RM0SBR, SparkFun-Electromechanical:DIP-8MM
- D10, D11, D12, D7, D8, D9: value MBRF1090 -> MBRF10H100
- R4: device SparkFun-Passives:1206 -> SparkFun-Resistors:0805
- moved R4 393.4 mm to (-200.0, -172.1), turned to 0 degrees
- moved U8 33.0 mm to (67.3, 55.9), flipped to the bottom, turned to 180 degrees
Connections:
- removed net !CS: MOD1.45
- removed net !FAULT: MOD1.49
- removed net !OCTW: MOD1.50
- removed net EN_GATE: MOD1.40
- removed net MISO: MOD1.47
- removed net MOSI: MOD1.46
- removed net SCLK: MOD1.48
- new net 15V1: D15.C
- new net 15V2: D16.C
- new net GND1: D15.A
- new net GND2: D16.A
- new net MODESET1: SW1.1
- new net MODESET2: SW1.2
- new net MODESET3: R61.1, SW1.4
- new net MODESET4: R62.1, SW1.8
- new net N$53: MOD2.3, R60.2
- new net N$54: MOD2.2, R59.2
- new net N$55: MOD2.6, R62.2
- new net VDD: MOD2.26
- new net VDDIO: MOD2.52
- net !VIN-FAULT: no longer MOD1.44
- net 15V: now also D14.C
- net 5V: now also C21.1, C22.1; no longer MOD1.26, MOD1.52
- net GND: now also C21.2, C22.2, D14.A, MOD2.1, MOD2.25, MOD2.51, SW1.C1, SW1.C2; no longer MOD1.1, MOD1.25, MOD1.51
- net INH_A: no longer MOD1.39
- net INH_B: no longer MOD1.37
- net INH_C: no longer MOD1.35
- net INL_A: no longer MOD1.38
- net INL_B: no longer MOD1.36
- net INL_C: no longer MOD1.34
- net ISENSE: no longer MOD1.3
- net N$16: no longer MOD1.30
- net N$30: now also MOD2.5, R61.2; no longer MOD1.24, SJ2.1
- net N$32: no longer MOD1.33
- net N$33: no longer MOD1.32
- net N$34: no longer MOD1.31
- net N$39: no longer MOD1.6
- net N$41: no longer MOD1.29
- net N$42: no longer MOD1.22
- net N$43: no longer MOD1.13
- net N$44: no longer MOD1.15
- net N$47: no longer MOD1.11
- net N$48: no longer MOD1.12
- net N$49: no longer MOD1.23
- net N$8: no longer MOD1.10
- net SCL: no longer MOD1.8
- net SDA: no longer MOD1.9
- net T_ALERT: no longer MOD1.21
- net VSENSE: no longer MOD1.2
Routing:
- net 5V: track 521.5 -> 4.03 mm, vias 12 -> 0
- net THROTTLE_2: track 219.7 -> 23.2 mm, vias 3 -> 1
- net H2: track 195.6 -> 0.35 mm, vias 5 -> 0
- net H1: track 189.8 -> 0.00 mm, vias 4 -> 0
- net H3: track 182.4 -> 0.00 mm, vias 6 -> 0
- net REVERSE: track 178.8 -> 0.00 mm, vias 2 -> 0
- net SCL: track 146.9 -> 0.00 mm, vias 4 -> 0
- net SDA: track 137.5 -> 0.00 mm, vias 4 -> 0
- net DISABLE: track 131.3 -> 0.00 mm, vias 3 -> 0
- net T_ALERT: track 111.4 -> 0.09 mm, vias 6 -> 0
- net GND: track 104.1 -> 10.6 mm, vias 79 -> 29
- net N$41: track 77.7 -> 0.00 mm, vias 2 -> 0
- net VSENSE: track 80.2 -> 5.52 mm, vias 2 -> 0
- net ISENSE: track 122.1 -> 51.0 mm, vias 3 -> 2
- net N$42: track 61.8 -> 0.00 mm, vias 2 -> 0
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- removed copper zone on layer 1, net 5V
- removed copper zone on layer 15, net KEEPOUT
- removed copper zone on layer 2, net KEEPOUT
- removed copper zone on layer 1, net PREJUMP_5V
