File: PCBs/Projects/MotorController/Main.brd (EAGLE design)
At the start: 172.7 x 99.1 mm, 155 parts, among them Q1 ZXMP10A17GQ, Q2 MMBT5551LT1G, Q3 BUK9240-100A.118, Q4 BUK9240-100A.118, Q5 NCV8440, Q7 NCV8440, SW1 DIP-SWTCH-16POSCD16RM0SBR, U1 LT8631, U11 LT4356-2, U12 UCC27211A-Q1, U13 UCC27211A-Q1, U14 UCC27211A-Q1, U2 ESDA6V1SC6Y, U3 ESDA6V1SC6Y, U4 ESDA6V1SC6Y, U5 TMP101, U6 ACS758LCB, U7 ESDA6V1SC6Y, U8 MTI85W100GC, U9 LT3045

Commit message: Added test points to schematic -Restarted board
Parts:
- removed MOD2: PSOC5LP-DEVBRDCY8CKIT-059, modules:CYKIT059
- removed Q7: NCV8440, SparkFun-DiscreteSemi:SOT223
- removed U14: UCC27211A-Q1, IC:SOIC-8-EP
- added C35: 0.01u, SparkFun-Capacitors:0805
- added F1, F2: B59607A120A62, SparkFun-PowerIC:1210
- added MOD1: PSOC5LP-DEVBRDCY8CKIT-059, modules:CYKIT059
- added Q6: NCV8440, SparkFun-DiscreteSemi:SOT223
- added TP1, TP10, TP11, TP12, TP13, TP14, TP15, TP16, TP17, TP2, TP3, TP4, TP5, TP6, TP7, TP8, TP9: (no value), SparkFun-Passives:TEST-POINT-MINI
- added U10: UCC27211A-Q1, IC:SOIC-8-EP
- C10: value 2.2u -> 5600p
- C12: value 4.7u -> 4.7; device SparkFun-Capacitors:1210 -> SparkFun-Capacitors:EIA3216
- C14: value 5600p -> DNP; device SparkFun-Capacitors:1210 -> SparkFun-Capacitors:0805
- C16: value 47u -> 10u
- C18: value 10u -> 47u
- C19: value 10u -> 0.1u; device SparkFun-Capacitors:1210 -> SparkFun-Capacitors:0805
- C20: value DNP -> 0.1u
- C23, C24, C25, C8: value 0.1u -> 0.01u
- C27, C31: value 0.01u -> 0.1u
- C28, C29: value 0.01u -> 4.7u; device SparkFun-Capacitors:0805 -> SparkFun-Capacitors:1210
- C30: value 0.1u -> 4.7u; device SparkFun-Capacitors:0805 -> SparkFun-Capacitors:1210
- C32: value 4.7 -> 0.1u; device SparkFun-Capacitors:EIA3216 -> SparkFun-Capacitors:0805
- C33, C6: value 4.7u -> 0.1u; device SparkFun-Capacitors:1210 -> SparkFun-Capacitors:0805
- C5: value 0.1u -> 2.2u; device SparkFun-Capacitors:0805 -> SparkFun-Capacitors:1210
- C7: value 2.2u -> 10u
- C9: value 0.01u -> 2.2u; device SparkFun-Capacitors:0805 -> SparkFun-Capacitors:1210
- D10, D8, D9: value MBRF10H100 -> 1SMA15AT3G; device SparkFun-DiscreteSemi:TO220V_2 -> SparkFun-DiscreteSemi:SMA-DIODE
- D13: value GREEN -> MBRF10H100; device SparkFun-LED:LED-1206 -> SparkFun-DiscreteSemi:TO220V_2
- D14, D15, D16: value 1SMA15AT3G -> MBRF10H100; device SparkFun-DiscreteSemi:SMA-DIODE -> SparkFun-DiscreteSemi:TO220V_2
- D6: value CLV1A-FKB -> GREEN; device SparkFun-LED:P-LCC-4-3 -> SparkFun-LED:LED-1206
- D7: value MBRF10H100 -> CLV1A-FKB; device SparkFun-DiscreteSemi:TO220V_2 -> SparkFun-LED:P-LCC-4-3
- R11: value 4.99k -> 274k
- R12: value 274k -> 4.99k
- R13: value 124k -> 10
- R14: value 10k -> 0.5
- R15: value 499 -> 2; device SparkFun-Resistors:0805 -> SparkFun-Passives:1206
- R16: value 25.5k -> 124k
- R17: value 1M -> 10k
- R18: value 57.6k -> 47k
- R19: value 2.7k -> 25.5k
- R20: value 100 -> 499
- R21: value 100 -> 47k
- R22: value 100 -> 1M
- R23: value 100 -> 57.6k
- R24, R57: value 1k -> 10
- R25: value 1k -> 140k
- R26: value 1k -> 10k
- R27: value 100 -> 2.7k
- R28: value 100 -> 1k
- R33: value 510k -> 4.7k
- R34, R35: value 1k -> 100
- R36, R37: value 4.7k -> 100
- R38, R39, R40: value 10k -> 100
- R41: value 100k -> 100; device SparkFun-Resistors:1206 -> SparkFun-Resistors:0805
- R42: value 5.1k -> 1k; device SparkFun-Resistors:1206 -> SparkFun-Resistors:0805
- R43, R44: value 10 -> 1k
- R45, R47: value 10 -> 100
- R46: value 10 -> 4.7k
- R48: value 10 -> 100k; device SparkFun-Resistors:0805 -> SparkFun-Resistors:1206
- R49: value 1M -> 5.1k
- R50: value 10 -> 10k
- R51: value 0.5 -> 10k
- R52: value 47k -> 10k
- R53: value 10 -> 510k
- R54: value 140k -> 1k
- R55: value 10k -> 1k
- R56: value 2 -> 10; device SparkFun-Passives:1206 -> SparkFun-Resistors:0805
- R58: value 47k -> 10
- R59, R60, R61: value 100 -> 10
- R62: value 100 -> 1M; device SparkFun-Resistors:0805 -> SparkFun-Resistors:1206
- R8: value 0.016 -> 0.2
- U1: value LT8631 -> LT4356-2; device IC:TSSOP-20-FE -> IC:SOIC-16
- U11: value LT4356-2 -> UCC27211A-Q1; device IC:SOIC-16 -> IC:SOIC-8-EP
- U13: value UCC27211A-Q1 -> MTI85W100GC; device IC:SOIC-8-EP -> IC:ISOPLUS-DIL
- U2: value ESDA6V1SC6Y -> LT8631; device IC:SOT23-6 -> IC:TSSOP-20-FE
- U3: value ESDA6V1SC6Y -> LT3045; device IC:SOT23-6 -> IC:MSOP-12-EP
- U4: value ESDA6V1SC6Y -> TMP101; device IC:SOT23-6 -> SparkFun-DigitalIC:SOT23-6
- U5: value TMP101 -> ACS758LCB; device SparkFun-DigitalIC:SOT23-6 -> IC:CB5PIN
- U6: value ACS758LCB -> ESDA6V1SC6Y; device IC:CB5PIN -> IC:SOT23-6
- U8: value MTI85W100GC -> ESDA6V1SC6Y; device IC:ISOPLUS-DIL -> IC:SOT23-6
- U9: value LT3045 -> ESDA6V1SC6Y; device IC:MSOP-12-EP -> IC:SOT23-6
- moved FD6 344.8 mm to (-116.8, 153.7)
- moved FD5 343.0 mm to (-114.3, 153.7)
- moved FD4 341.2 mm to (-111.8, 153.7)
- moved R59 334.1 mm to (-61.0, 151.1)
- moved R60 333.9 mm to (-64.8, 151.1)
- moved R61 333.6 mm to (-68.6, 151.1)
- moved D14 331.5 mm to (-38.1, 127.0)
- moved D15 328.0 mm to (-53.3, 127.0)
- moved R4 327.5 mm to (-108.0, 142.2)
- moved D16 325.3 mm to (-68.6, 127.0)
- moved C21 324.7 mm to (-102.9, 151.1)
- moved C22 324.6 mm to (-106.7, 151.1)
- moved R62 317.5 mm to (-95.2, 142.2)
- moved R58 315.8 mm to (-57.1, 151.1)
- moved R57 305.6 mm to (-53.3, 151.1)
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Connections:
- removed net N$41 (its old number): R22.2
- removed net N$49 (its old number): R21.2
- new net N$47: R39.2
- new net N$48: R40.2
- new net N$56: F1.2, J4.1
- new net N$57: C34.1, F2.1, J5.5
- net !VIN-FAULT: now also U1.10; no longer U11.10
- net 15V: now also C18.1, C28.1, C29.1, C30.1, D10.C, R15.1, R21.2, R22.2, R27.2, R28.2, TP3.P$1, U10.1, U11.1, U2.12; no longer C16.1, C33.1, C4.1, C6.1, D14.C, R17.2, R19.2, R52.2, R56.1, R57.2, U1.12, U13.1, U14.1
- net 15V1: now also D9.C; no longer D15.C
- net 15V2: now also D8.C; no longer D16.C
- net 15V_PG: now also R21.1, U2.5, U3.4; no longer R52.1, U1.5, U9.4
- net 5V: now also C16.1, C20.1, C23.1, D7.2, F1.1, F2.2, R18.2, R25.1, R33.1, R46.1, R50.1, R51.1, R52.1, TP2.P$1, U3.10, U3.11, U3.12, U4.4, U5.1, U9.1; no longer C22.1, C28.1, C30.1, D6.2, J4.1, J5.5, R34.1, R36.1, R37.1, R38.1, R39.1, R40.1, R58.2, U5.4, U6.1, U7.1, U9.10, U9.11, U9.12
- net 5V_PG: now also Q6.1, R18.1, U3.5; no longer Q7.1, R58.1, U9.5
- net 5V_SET_CONNECTION: now also C12.A, R24.1, U3.8; no longer C32.A, R53.1, U9.8
- net A: now also C31.2, D11.2, D12.1, U10.4, U13.L1, U13.S1; no longer C5.2, D7.2, D8.1, U12.4, U8.L1, U8.S1
- net B: now also C32.2, D13.2, D14.1, U11.4, U13.L2, U13.S3; no longer C23.2, D10.1, D9.2, U13.4, U8.L2, U8.S3
- net C: now also C33.2, D15.2, D16.1, U12.4, U13.L3, U13.S5; no longer C34.2, D11.2, D12.1, U14.4, U8.L3, U8.S5
- net DISABLE: now also R45.1, U6.6; no longer R23.1, U2.6
- net DISP_OUT: now also R31.1, U8.4; no longer R22.1, U4.4
- net FB: now also R11.1, R12.2, U1.2; no longer R11.2, R12.1, U11.2
- net GATEDRV: now also U1.5; no longer U11.5
- net GH_A: now also R56.2, TP17.P$1, U10.3; no longer R43.2, U12.3
- net GH_B: now also R58.2, TP15.P$1, U11.3; no longer R45.2, U13.3
- net GH_C: now also R60.2, TP13.P$1, U12.3; no longer R47.2, U14.3
- net GL_A: now also R57.2, TP16.P$1, U10.8; no longer R44.2, U12.8
- net GL_B: now also R59.2, TP14.P$1, U11.8; no longer R46.2, U13.8
- net GL_C: now also R61.2, TP12.P$1, U12.8; no longer R48.2, U14.8
- net GND: now also C12.C, C27.2, C28.2, C34.2, C35.2, C7.2, C8.2, D10.A, D14.2, D16.2, MOD1.1, MOD1.25, MOD1.51, Q6.3, R12.1, R13.1, R17.1, R19.1, R20.2, R23.1, R24.2, R26.2, R62.1, U1.12, U10.7, U10.EP1, U10.EP2, U10.EP3, U10.EP4, U10.EP5, U10.EP6, U10.EXP, U11.7, U11.EP1, U11.EP2, U11.EP3, U11.EP4, U11.EP5, U11.EP6, U11.EXP, U13.L-, U13.S2, U13.S4, U13.S6, U2.13, U2.15, U2.6, U2.7, U2.9, U2.EXP, U3.9, U3.EXP, U6.5, U8.2, U8.5, U9.2, U9.5; no longer C11.2, C24.2, C31.2, C32.C, C33.2, C4.2, D10.2, D14.A, D8.2, MOD2.1, MOD2.25, MOD2.51, Q7.3, R11.1, R15.2, R16.1, R18.1, R33.2, R35.2, R42.1, R50.1, R51.1, U1.13, U1.15, U1.6, U1.7, U1.9, U1.EXP, U11.12, U13.7, U13.EP1, U13.EP2, U13.EP3, U13.EP4, U13.EP5, U13.EP6, U13.EXP, U14.7, U14.EP1, U14.EP2, U14.EP3, U14.EP4, U14.EP5, U14.EP6, U14.EXP, U2.2, U2.5, U3.2, U3.5, U5.5, U8.L-, U8.S2, U8.S4, U8.S6, U9.9, U9.EXP
- net GND1: now also D9.A; no longer D15.A
- net GND2: now also D8.A; no longer D16.A
- net GPIO_TBD: now also R41.1, U8.6; no longer R20.1, U4.6
- net H1: now also C23.2, R38.1, R50.2, TP6.P$1, U9.3; no longer C26.2, R28.1, R38.2, U7.3
- net H2: now also C24.2, R39.1, R51.2, TP7.P$1, U9.4; no longer C27.2, R29.1, R39.2, U7.4
- net H3: now also C26.2, R40.1, R52.2, TP8.P$1, U9.6; no longer C28.2, R30.1, R40.2, U7.6
- net ILIMIT_5V: now also R20.1, U3.6; no longer R15.1, U9.6
- net INH_A: now also U10.5; no longer U12.5
- net INH_B: now also U11.5; no longer U13.5
- net INH_C: now also U12.5; no longer U14.5
- net INL_A: now also U10.6; no longer U12.6
- net INL_B: now also U11.6; no longer U13.6
- net INL_C: now also U12.6; no longer U14.6
- net ISENSE: now also C25.1, TP10.P$1, U5.3, U7.4; no longer C29.1, U3.4, U6.3
- net MODESET3: now also R36.1; no longer R61.1
- net MODESET4: now also R37.1; no longer R62.1
- net MONITOR_RX: now also R30.1, U8.3; no longer R32.1, U4.3
- net MONITOR_TX: now also R29.1, U8.1; no longer R31.1, U4.1
- net N$1: now also U1.1; no longer U11.1
- net N$10: now also U2.14; no longer U1.14
- net N$12: now also C11.1, U2.18; no longer C8.1, U1.18
- net N$13: now also U1.16; no longer U11.16
- net N$14: now also C8.1, R16.1, R17.2, U2.3; no longer C9.1, R13.1, R14.2, U1.3
- net N$15: now also C9.1, U2.16; no longer C10.1, U1.16
- net N$16: now also R45.2; no longer R23.2
- net N$17: now also R19.2, U2.8; no longer R16.2, U1.8
- net N$18: now also C10.1, U2.10; no longer C14.1, U1.10
- net N$2: now also C31.1, U10.2; no longer C5.1, U12.2
- net N$21: now also C14.1, R22.1, R23.2, U2.11; no longer C20.1, R17.1, R18.2, U1.11
- net N$24: now also C7.1, R15.2, U3.1, U3.2, U3.3; no longer C18.1, R56.2, U9.1, U9.2, U9.3
- net N$25: now also C4.2, R13.2; no longer C12.2, R50.2
- net N$26: now also C5.2, R14.2; no longer C7.2, R51.2
- net N$27: now also R58.1, U13.G3; no longer R45.1, U8.G3
- net N$28: now also R56.1, U13.G1; no longer R43.1, U8.G1
- net N$3: now also C32.1, U11.2; no longer C23.1, U13.2
- net N$30: now also MOD1.5, R36.2; no longer MOD2.5, R61.2
- net N$31: now also C35.1, R62.2; no longer C31.1, R49.2
- net N$32: now also R44.1; no longer R26.1
- net N$33: now also R43.1; no longer R25.1
- net N$34: now also R42.1; no longer R24.1
- net N$35: now also D7.1, R44.2; no longer D6.1, R26.2
- net N$36: now also D7.4, R43.2; no longer D6.4, R25.2
- net N$37: now also D7.3, R42.2; no longer D6.3, R24.2
- net N$38: now also R57.1, U13.G2; no longer R44.1, U8.G2
- net N$39: now also C22.1, R47.2, TP11.P$1; no longer C25.1, R27.2
- net N$40: now also R27.1; no longer R19.1
- net N$42: now also R41.2; no longer R20.2
- net N$45: now also D6.A, R28.1; no longer D13.A, R57.1
- net N$46: now also D6.C, Q6.2, Q6.4; no longer D13.C, Q7.2, Q7.4
- net N$5: now also C33.1, U12.2; no longer C34.1, U14.2
- net N$50: now also R59.1, U13.G4; no longer R46.1, U8.G4
- net N$51: now also R60.1, U13.G5; no longer R47.1, U8.G5
- net N$52: now also R61.1, U13.G6; no longer R48.1, U8.G6
- net N$53: now also MOD1.3, R35.2; no longer MOD2.3, R60.2
- net N$54: now also MOD1.2, R34.2; no longer MOD2.2, R59.2
- net N$55: now also MOD1.6, R37.2; no longer MOD2.6, R62.2
- net N$6: now also C11.2, U2.20; no longer C8.2, U1.20
- net N$8: now also R38.2; no longer R28.2
- net PG_FB: now also R25.2, R26.1, U3.7; no longer R54.2, R55.1, U9.7
- net POST-SENSE: now also U1.7; no longer U11.7
- net PRE-SENSE: now also U1.8, U1.9; no longer U11.8, U11.9
- net REVERSE: now also R32.1, U6.4; no longer R21.1, U2.4
- net SCL: now also R33.2, TP4.P$1, U4.1; no longer R36.2, U5.1
- net SDA: now also R46.2, TP5.P$1, U4.6; no longer R37.2, U5.6
- net THROTTLE_1: now also R54.2, U6.1; no longer R34.2, U2.1
- net THROTTLE_2: now also R47.1, R53.1, U6.3; no longer R27.1, R33.1, U2.3
- net THROTTLE_3: now also R55.1; no longer R35.1
- net T_ALERT: now also U4.3; no longer U5.3
- net UNDERVOLTAGE: now also U1.14; no longer U11.14
- net VCC: now also C4.1, C5.1, C6.1, R11.2, R16.2, R48.2, TP1.P$1, U1.4, U2.1; no longer C11.1, C12.1, C7.1, R12.2, R13.2, R41.2, U1.1, U11.4
- net VDD: now also MOD1.26; no longer MOD2.26
- net VDDIO: now also MOD1.52; no longer MOD2.52
- net VIN: now also U5.4_1, U5.4_2, U5.4_3, U5.4_4, U5.4_5, U5.4_6, U5.4_7, U5.4_8; no longer U6.4_1, U6.4_2, U6.4_3, U6.4_4, U6.4_5, U6.4_6, U6.4_7, U6.4_8
- net VSENSE: now also R48.1, R49.2, U7.1; no longer R41.1, R42.2, U3.1
- net V_BATT: now also D13.1, D15.1, U13.L+, U5.5_1, U5.5_2, U5.5_3, U5.5_4, U5.5_5, U5.5_6, U5.5_7, U5.5_8; no longer D7.1, D9.1, U6.5_1, U6.5_2, U6.5_3, U6.5_4, U6.5_5, U6.5_6, U6.5_7, U6.5_8, U8.L+
Routing:
- net ISENSE: track 51.0 -> 0.00 mm, vias 2 -> 0
- net N$13: track 32.0 -> 0.00 mm, vias 2 -> 0
- net GATEDRV: track 24.6 -> 0.00 mm, vias 2 -> 0
- net PRE-SENSE: track 23.5 -> 0.00 mm, vias 2 -> 0
- net THROTTLE_2: track 23.2 -> 0.00 mm, vias 1 -> 0
- net THROTTLE_1: track 19.2 -> 0.00 mm
- net V_BATT: track 18.4 -> 0.00 mm, vias 26 -> 0
- net UNDERVOLTAGE: track 15.4 -> 0.00 mm, vias 2 -> 0
- net N$22: track 13.4 -> 0.00 mm
- net THROTTLE_3: track 13.1 -> 0.00 mm
- net VCC: track 12.3 -> 0.00 mm, vias 4 -> 0
- net GND: track 10.6 -> 0.00 mm, vias 29 -> 0
- net N$31: track 9.89 -> 0.00 mm
- net N$19: track 7.39 -> 0.00 mm
- net POST-SENSE: track 6.56 -> 0.00 mm, vias 1 -> 0
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- removed copper zone on layer 1, net A
- removed copper zone on layer 2, net A
- removed copper zone on layer 1, net B
- removed copper zone on layer 2, net B
- removed copper zone on layer 1, net C
- removed copper zone on layer 2, net C
- removed copper zone on layer 1, net GND
- removed copper zone on layer 15, net GND
- removed copper zone on layer 16, net GND
- removed copper zone on layer 2, net GND
- removed copper zone on layer 1, net IND_LOOP_IN
- removed copper zone on layer 15, net IND_LOOP_IN
- removed copper zone on layer 16, net IND_LOOP_IN
- removed copper zone on layer 1, net IND_LOOP_OUT
- removed copper zone on layer 1, net POST-SENSE
- removed copper zone on layer 1, net PRE-SENSE
- removed copper zone on layer 1, net VCC
- removed copper zone on layer 16, net VCC
- removed copper zone on layer 1, net VIN
- removed copper zone on layer 16, net VIN
- removed copper zone on layer 2, net VIN
- removed copper zone on layer 1, net V_BATT
- removed copper zone on layer 16, net V_BATT
- removed copper zone on layer 2, net V_BATT
Other:
- board size 172.7 x 99.1 mm -> 160 x 94 mm
- board text removed: ""Don't forget the heatshrink!""
- board text removed: "+"
- board text removed: "-"
- board text removed: "1"
- board text removed: "2"
- board text removed: "3"
- board text removed: "4"
- board text removed: "5v"
- board text removed: "60V MAX"
- board text removed: "A"
- board text removed: "B"
- board text removed: "BLDC Controller Rev B"
- board text removed: "C"
- board text removed: "D"
- board text removed: "DANGER\! HIGH VOLTAGES PRESENT ON BOARD"
- board text removed: "DO"
- board text removed: "Engineer: Tom D'Agostino"
- board text removed: "Fabrication Notes: 1: The milling layer denotes internal cutouts. 2: Internal cutouts are not plated."
- board text removed: "GND"
- board text removed: "H1"
- board text removed: "H2"
- board text removed: "H3"
- board text removed: "IO"
- board text removed: "R"
- board text removed: "RX"
- board text removed: "S E M"
- board text removed: "Saint Thomas Academy Experimental Vehicle Team"
- board text removed: "T1"
- board text removed: "T2"
- board text removed: "T3"
- board text removed: "TX"

Commit message: switching psu layout 50% done
Parts:
- removed C35: 0.01u, SparkFun-Capacitors:0805
- C10: value 5600p -> 0.1u; device SparkFun-Capacitors:1210 -> SparkFun-Capacitors:0805
- C11: value 0.1u -> 4.7; device SparkFun-Capacitors:0805 -> SparkFun-Capacitors:EIA3216
- C12: value 4.7 -> 200p; device SparkFun-Capacitors:EIA3216 -> SparkFun-Capacitors:0805
- C13: value 200p -> DNP
- C14: value DNP -> 47u; device SparkFun-Capacitors:0805 -> SparkFun-Capacitors:1210
- C15: value 47u -> 10u
- C16: value 10u -> 47u
- C18: value 47u -> 0.1u; device SparkFun-Capacitors:1210 -> SparkFun-Capacitors:0805
- C22, C34: value 0.1u -> 0.01u
- C26: value 0.01u -> 0.1u
- C27: value 0.1u -> 4.7u; device SparkFun-Capacitors:0805 -> SparkFun-Capacitors:1210
- C3: device SparkFun-Passives:1210 -> SparkFun-Capacitors:1210
- C30: value 4.7u -> 0.1u; device SparkFun-Capacitors:1210 -> SparkFun-Capacitors:0805
- C4: value 4.7u -> 2.2u
- C5: value 2.2u -> 0.1u; device SparkFun-Capacitors:1210 -> SparkFun-Capacitors:0805
- C6: value 0.1u -> 10u; device SparkFun-Capacitors:0805 -> SparkFun-Capacitors:1210
- C7: value 10u -> 0.01u; device SparkFun-Capacitors:1210 -> SparkFun-Capacitors:0805
- C8: value 0.01u -> 2.2u
- C9: value 2.2u -> 5600p; device SparkFun-Capacitors:1210 -> SparkFun-Capacitors:0805
- R8: device SparkFun-Resistors:R2010 -> SparkFun-Resistors:1206
- moved R9 231.7 mm to (95.5, 65.8), turned to 180 degrees
- moved R10 231.3 mm to (91.7, 66.8), turned to 90 degrees
- moved R11 230.6 mm to (89.2, 73.2), turned to 270 degrees
- moved R7 228.0 mm to (101.9, 87.1), turned to 270 degrees
- moved R6 225.3 mm to (101.9, 83.3), turned to 270 degrees
- moved R5 224.1 mm to (99.3, 66.8), turned to 90 degrees
- moved R4 220.7 mm to (97.5, 61.7)
- moved D2 218.8 mm to (103.4, 61.7)
- moved D3 216.1 mm to (91.7, 61.7), turned to 180 degrees
- moved R3 215.4 mm to (104.1, 87.1), turned to 90 degrees
- moved U1 215.0 mm to (83.6, 78.0), turned to 90 degrees
- moved S3 214.2 mm to (129.5, 12.7)
- moved R2 212.8 mm to (104.1, 83.3), turned to 270 degrees
- moved Q1 196.9 mm to (109.7, 84.3), turned to 270 degrees
- moved R1 190.0 mm to (103.1, 91.4)
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Connections:
- removed net 15V1: D9.C
- removed net 15V2: D8.C
- removed net GND1: D9.A
- removed net GND2: D8.A
- removed net VDD: MOD1.26
- removed net VDDIO: MOD1.52
- net !VIN-FAULT: now also MOD1.49
- net 15V: now also C12.1, C14.1, C16.1, C27.1, D8.C, D9.C; no longer C13.1, C15.1, C18.1, C30.1
- net 5V: now also C15.1, C18.1, C22.1, C25.1, MOD1.26, MOD1.52; no longer C16.1, C21.1, C24.1, C27.1
- net 5V_SET_CONNECTION: now also C11.A; no longer C12.A
- net A: now also C30.2; no longer C31.2
- net B: now also C31.2; no longer C32.2
- net C: now also C32.2; no longer C33.2
- net GND: now also C11.C, C13.2, C24.2, C26.2, C33.2, C5.2, D8.A, D9.A; no longer C10.2, C12.C, C22.2, C25.2, C3.2, C30.2, C35.2
- net H1: now also C22.2; no longer C23.2
- net H2: now also C23.2; no longer C24.2
- net H3: now also C25.2; no longer C26.2
- net INH_A: now also MOD1.30
- net INH_B: now also MOD1.32
- net INH_C: now also MOD1.34
- net INL_A: now also MOD1.31
- net INL_B: now also MOD1.33
- net INL_C: now also MOD1.35
- net ISENSE: now also C24.1, MOD1.21; no longer C25.1
- net MODESET1: now also R34.1
- net MODESET2: now also R35.1
- net N$12: now also C10.1; no longer C11.1
- net N$14: now also C7.1; no longer C8.1
- net N$15: now also C8.1; no longer C9.1
- net N$16: now also MOD1.13
- net N$18: now also C9.1; no longer C10.1
- net N$2: now also C30.1; no longer C31.1
- net N$21: now also C12.2, C13.1; no longer C13.2, C14.1
- net N$24: now also C6.1; no longer C7.1
- net N$25: now also C3.2; no longer C4.2
- net N$26: now also C4.2; no longer C5.2
- net N$3: now also C31.1; no longer C32.1
- net N$31: now also C34.1; no longer C35.1
- net N$32: now also MOD1.36
- net N$33: now also MOD1.37
- net N$34: now also MOD1.38
- net N$39: now also C21.1, MOD1.7; no longer C22.1
- net N$41: now also MOD1.50
- net N$42: now also MOD1.39
- net N$43: now also MOD1.47
- net N$44: now also MOD1.48
- net N$47: now also MOD1.41
- net N$48: now also MOD1.40
- net N$49: now also MOD1.27
- net N$5: now also C32.1; no longer C33.1
- net N$57: now also C33.1; no longer C34.1
- net N$6: now also C10.2; no longer C11.2
- net N$8: now also MOD1.42
- net SCL: now also MOD1.11
- net SDA: now also MOD1.10
- net T_ALERT: now also MOD1.12
- net VCC: no longer C6.1
- net VSENSE: now also MOD1.17, TP9.P$1
Routing:
- net N$13: track 0.00 -> 36.0 mm, vias 0 -> 2
- net UNDERVOLTAGE: track 0.00 -> 34.3 mm, vias 0 -> 2
- net GATEDRV: track 0.00 -> 23.2 mm, vias 0 -> 2
- net VCC: track 0.00 -> 20.1 mm, vias 0 -> 13
- net N$14: track 0.00 -> 19.5 mm, vias 0 -> 3
- net PRE-SENSE: track 0.00 -> 18.8 mm
- net N$22: track 0.00 -> 13.0 mm
- net POST-SENSE: track 0.00 -> 10.7 mm
- net N$9: track 0.00 -> 8.04 mm
- net N$21: track 0.00 -> 6.40 mm
- net 15V: track 0.00 -> 6.02 mm
- net N$20: track 0.00 -> 5.53 mm
- net FB: track 0.00 -> 4.80 mm
- net N$19: track 0.00 -> 4.67 mm
- net N$4: track 0.00 -> 4.36 mm
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- added copper zone on layer 2, net GND
- added copper zone on layer 3, net GND
- added copper zone on layer 1, net N$10
- added copper zone on layer 1, net N$6
- added copper zone on layer 1, net POST-SENSE
- added copper zone on layer 1, net PRE-SENSE
- added copper zone on layer 1, net VCC
- added copper zone on layer 16, net VCC

Commit message: LDO placed and routed
Parts:
- R24: value 10 -> 49.9k
- moved D12 292.1 mm to (128.9, -25.4)
- moved D11 289.5 mm to (142.2, -23.5)
- moved C26 245.9 mm to (116.2, 89.8)
- moved D16 238.6 mm to (128.9, -6.99)
- moved D15 231.8 mm to (132.1, -12.1)
- moved TP1 227.3 mm to (81.0, 65.2)
- moved J4 215.8 mm to (67.9, 4.45), turned to 180 degrees
- moved D13 205.6 mm to (122.6, -18.4)
- moved TP3 205.4 mm to (56.3, 72.3)
- moved D14 204.7 mm to (114.9, -8.89)
- moved TP2 199.4 mm to (40.4, 78.9)
- moved C24 190.5 mm to (19.1, 18.9), turned to 180 degrees
- moved U12 187.8 mm to (66.0, 34.9), turned to 180 degrees
- moved R61 183.3 mm to (70.5, 31.8), turned to 90 degrees
- moved R60 177.9 mm to (70.5, 35.6), turned to 90 degrees
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Connections:
- net 15V: no longer R28.2
- net 5V: now also R28.2
Routing:
- net 15V_PG: track 0.00 -> 69.3 mm, vias 0 -> 5
- net 5V_PG: track 0.00 -> 36.7 mm, vias 0 -> 3
- net 5V: track 0.00 -> 25.8 mm
- net PG_FB: track 0.00 -> 15.6 mm, vias 0 -> 2
- net N$40: track 0.00 -> 12.6 mm, vias 0 -> 2
- net 15V: track 6.02 -> 18.3 mm
- net N$29: track 0.00 -> 11.1 mm
- net N$46: track 0.00 -> 10.9 mm
- net N$24: track 0.00 -> 9.77 mm
- net 5V_SET_CONNECTION: track 0.00 -> 4.71 mm
- net ILIMIT_5V: track 0.00 -> 2.33 mm
- net N$45: track 0.00 -> 2.05 mm
- net GND: track 0.00 -> 1.40 mm, vias 9 -> 104
- net N$14: track 19.5 -> 20.1 mm
- added copper zone on layer 1, net 15V
- added copper zone on layer 1, net 5V
- added copper zone on layer 1, net GND

Commit message: Major layout work
Parts:
- D10, D8, D9: value 1SMA15AT3G -> SZMM3Z18VST1G; device SparkFun-DiscreteSemi:SMA-DIODE -> SparkFun-DiscreteSemi:SOD-323
- moved U9 282.8 mm to (121.8, 4.95)
- moved C25 278.6 mm to (111.1, 4.45), turned to 90 degrees
- moved C23 266.9 mm to (111.1, 8.26), turned to 90 degrees
- moved C22 259.5 mm to (108.6, 12.1), turned to 90 degrees
- moved F2 259.2 mm to (136.3, 5.33), turned to 180 degrees
- moved C19 257.6 mm to (91.4, -22.2)
- moved C20 257.6 mm to (87.6, -22.2)
- moved C21 257.6 mm to (83.8, -22.2)
- moved FD1 257.6 mm to (86.4, -19.7)
- moved FD2 257.6 mm to (83.8, -19.7)
- moved FD3 257.6 mm to (81.3, -19.7)
- moved FD4 257.6 mm to (78.7, -19.7)
- moved FD5 257.6 mm to (76.2, -19.7)
- moved FD6 257.6 mm to (73.7, -19.7)
- moved FRAME1 257.6 mm to (71.1, -19.7)
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Connections:
- net INH_A: now also MOD1.39; no longer MOD1.30
- net INH_B: now also MOD1.37; no longer MOD1.32
- net INH_C: now also MOD1.35; no longer MOD1.34
- net INL_A: now also MOD1.38; no longer MOD1.31
- net INL_B: now also MOD1.36; no longer MOD1.33
- net INL_C: no longer MOD1.35
- net N$32: now also MOD1.33; no longer MOD1.36
- net N$33: now also MOD1.32; no longer MOD1.37
- net N$34: now also MOD1.31; no longer MOD1.38
- net N$42: now also MOD1.30; no longer MOD1.39
Routing:
- net 5V: track 25.8 -> 166.7 mm, vias 0 -> 7
- net H1: track 0.00 -> 48.2 mm
- net H2: track 0.00 -> 47.7 mm, vias 0 -> 1
- net H3: track 0.00 -> 45.1 mm, vias 0 -> 2
- net B: track 0.00 -> 21.5 mm, vias 0 -> 32
- net A: track 0.00 -> 21.4 mm, vias 0 -> 46
- net C: track 0.00 -> 21.4 mm, vias 0 -> 61
- net GH_C: track 0.00 -> 13.6 mm
- net GH_B: track 0.00 -> 13.6 mm
- net GH_A: track 0.00 -> 13.6 mm
- net N$40: track 12.6 -> 2.10 mm, vias 2 -> 0
- net GL_B: track 0.00 -> 7.03 mm
- net GL_C: track 0.00 -> 7.03 mm
- net GL_A: track 0.00 -> 6.98 mm
- net N$57: track 0.00 -> 6.58 mm
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- added copper zone on layer 3, net 15V
- added copper zone on layer 1, net A
- added copper zone on layer 16, net A
- added copper zone on layer 1, net B
- added copper zone on layer 16, net B
- added copper zone on layer 1, net C
- added copper zone on layer 16, net C
- added copper zone on layer 16, net GND
- added copper zone on layer 16, net N$2
- added copper zone on layer 16, net N$3
- added copper zone on layer 16, net N$5
- added copper zone on layer 1, net VIN
- added copper zone on layer 16, net VIN
- added copper zone on layer 2, net VIN
- added copper zone on layer 3, net VIN
- added copper zone on layer 1, net V_BATT
- added copper zone on layer 16, net V_BATT
- added copper zone on layer 2, net V_BATT
- added copper zone on layer 3, net V_BATT
- removed copper zone on layer 2, net GND
- removed copper zone on layer 3, net GND

Commit message: More signals run
Parts:
- moved R54 141.8 mm to (134.0, 91.8)
- moved R55 129.3 mm to (136.5, 79.4), turned to 180 degrees
- moved C19 105.0 mm to (45.1, 72.0), turned to 90 degrees
- moved C21 92.2 mm to (33.4, 55.0), turned to 270 degrees
- moved U7 82.9 mm to (34.9, 27.3)
- moved TP8 74.2 mm to (104.6, 5.33)
- moved TP7 73.1 mm to (104.6, 9.14)
- moved TP6 72.5 mm to (104.6, 13.0)
- moved TP4 69.5 mm to (87.6, 19.1)
- moved TP5 69.5 mm to (87.6, 21.6)
- moved R53 67.1 mm to (38.7, 55.0), turned to 270 degrees
- moved C20 61.8 mm to (33.0, 6.73), turned to 270 degrees
- moved R42 38.9 mm to (61.0, 1.27)
- moved R43 36.5 mm to (64.8, 3.81)
- moved R44 26.5 mm to (57.1, 7.62), turned to 0 degrees
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Connections:
- net INL_C: now also MOD1.34
- net REVERSE: now also U6.3; no longer U6.4
- net THROTTLE_2: now also U6.4; no longer U6.3
- net VSENSE: now also U7.3; no longer U7.1
Routing:
- net DISABLE: track 0.00 -> 160.3 mm, vias 0 -> 3
- net THROTTLE_2: track 0.00 -> 150.5 mm, vias 0 -> 4
- net 5V: track 166.7 -> 303.6 mm, vias 7 -> 9
- net INL_A: track 0.00 -> 26.4 mm
- net INL_B: track 0.00 -> 20.6 mm
- net INH_A: track 0.00 -> 19.2 mm
- net THROTTLE_1: track 0.00 -> 16.1 mm
- net INL_C: track 0.00 -> 15.5 mm
- net INH_B: track 0.00 -> 13.7 mm
- net N$39: track 0.00 -> 12.4 mm
- net REVERSE: track 0.00 -> 12.3 mm, vias 0 -> 1
- net THROTTLE_3: track 0.00 -> 11.5 mm
- net INH_C: track 0.00 -> 9.18 mm
- net N$53: track 0.00 -> 5.58 mm
- net N$30: track 0.00 -> 5.58 mm
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
Commit message: Most Layout complete
Parts:
- moved FD2 134.1 mm to (5.08, 88.9), flipped to the bottom
- moved FD5 129.8 mm to (5.08, 88.9)
- moved FD4 113.5 mm to (111.8, 88.9)
- moved FD1 111.5 mm to (111.8, 88.9), flipped to the bottom
- moved F1 89.1 mm to (78.7, 3.94), turned to 180 degrees
- moved J4 87.4 mm to (74.2, 3.94), turned to 180 degrees
- moved FD3 79.7 mm to (5.08, 3.81), flipped to the bottom
- moved FRAME1 73.8 mm to (0.00, 0.00)
- moved FD6 72.5 mm to (5.08, 3.81)
- moved FRAME2 71.3 mm to (0.00, 0.00)
- moved FRAME3 68.9 mm to (0.00, 0.00)
- moved FRAME4 66.5 mm to (0.00, 0.00)
- moved FRAME5 64.1 mm to (0.00, 0.00)
- moved FRAME6 61.6 mm to (0.00, 0.00)
- moved R62 60.6 mm to (5.84, 16.1), turned to 180 degrees
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Connections:
- net DISP_OUT: now also U8.6; no longer U8.4
- net GPIO_TBD: now also U8.4; no longer U8.6
- net MONITOR_RX: now also U8.1; no longer U8.3
- net MONITOR_TX: now also U8.3; no longer U8.1
- net N$35: now also D7.3; no longer D7.1
- net N$37: now also D7.1; no longer D7.3
Routing:
- net REVERSE: track 12.3 -> 194.5 mm, vias 1 -> 5
- net ISENSE: track 4.57 -> 185.2 mm, vias 0 -> 3
- net T_ALERT: track 0.00 -> 124.4 mm, vias 0 -> 3
- net VSENSE: track 2.41 -> 122.3 mm
- net SCL: track 0.00 -> 115.7 mm, vias 0 -> 2
- net 5V: track 303.6 -> 415.1 mm, vias 9 -> 14
- net SDA: track 0.00 -> 111.4 mm, vias 0 -> 4
- net DISP_OUT: track 0.00 -> 101.4 mm, vias 0 -> 3
- net MODESET1: track 0.00 -> 95.3 mm, vias 0 -> 2
- net H3: track 49.0 -> 142.2 mm, vias 2 -> 6
- net H2: track 51.7 -> 144.6 mm, vias 1 -> 4
- net GND: track 1.40 -> 94.1 mm, vias 148 -> 228
- net MONITOR_RX: track 0.00 -> 91.5 mm, vias 0 -> 2
- net H1: track 52.2 -> 142.8 mm, vias 0 -> 3
- net MONITOR_TX: track 0.00 -> 87.9 mm, vias 0 -> 3
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- added copper zone on layer 2, net GND
- added copper zone on layer 3, net GND
Other:
- board size 160 x 94 mm -> 144.8 x 94 mm

Commit message: Board mostly completed
Parts:
- D4: device SparkFun-DiscreteSemi:SMA-DIODE -> SparkFun-DiscreteSemi:SMA-DIODE-BI
- moved C22 2.54 mm to (95.2, 11.9)
- moved R50 2.54 mm to (92.7, 11.9)
- moved C18 2.18 mm to (73.4, 25.1), turned to 180 degrees
- moved TP2 0.25 mm to (24.5, 79.1)
- moved D4 0.18 mm to (83.3, 86.1), turned to 270 degrees
- moved R13 0.13 mm to (63.2, 72.9)
- moved TP13 0.13 mm to (45.1, 36.3)
- moved TP15 0.13 mm to (45.1, 48.4)
- moved TP17 0.13 mm to (45.1, 60.5)
- moved R7 0.13 mm to (86.0, 87.1)
- moved R20 0.10 mm to (36.4, 85.1)
- moved C2 0.10 mm to (69.7, 71.8)
- moved R19 0.08 mm to (61.5, 72.9)
- moved C6 0.05 mm to (36.4, 79.2)
Connections:
- net GND: now also D4.A; no longer D4.C
- net PRE-SENSE: now also D4.C; no longer D4.A
Routing:
- net GND: track 94.1 -> 103.1 mm, vias 228 -> 251
- net VSENSE: track 122.3 -> 130.9 mm, vias 0 -> 2
- net 5V: track 415.1 -> 410.7 mm, vias 14 -> 13
- net POST-SENSE: track 10.6 -> 14.9 mm
- net VCC: track 20.0 -> 17.6 mm
- net H3: track 142.2 -> 140.2 mm, vias 6 -> 5
- net ISENSE: track 185.2 -> 184.3 mm
- net 5V_PG: track 43.2 -> 43.8 mm
Other:
- board text added: "+"
- board text added: "-"
- board text added: "1"
- board text added: "2"
- board text added: "3"
- board text added: "4"
- board text added: "65v MAX"
- board text added: "A"
- board text added: "B"
- board text added: "BLDC Controller Rev C"
- board text added: "Board Number"
- board text added: "C"
- board text added: "DANGER\! HIGH VOLTAGES PRESENT ON BOARD"
- board text added: "Engineer: Tom D'Agostino"
- board text added: "SEM"
- board text added: "Saint Thomas Academy Experimental Vehicle Team"

Commit message: All DRC errors fixed, labels applied, teardrop ULP run
Routing:
- net GND: track 103.1 -> 162.7 mm, vias 251 -> 255
- net 5V: track 410.7 -> 470.0 mm
- net REVERSE: track 194.5 -> 241.3 mm
- net THROTTLE_2: track 153.4 -> 199.9 mm
- net H2: track 144.6 -> 178.0 mm
- net H3: track 140.2 -> 173.4 mm
- net MODESET2: track 74.4 -> 105.4 mm
- net MODESET4: track 67.8 -> 98.4 mm
- net H1: track 143.0 -> 172.0 mm
- net ISENSE: track 184.3 -> 212.5 mm
- net DISABLE: track 161.9 -> 188.6 mm
- net 15V_PG: track 64.6 -> 89.4 mm
- net SDA: track 111.4 -> 136.1 mm
- net MODESET3: track 81.8 -> 106.1 mm
- net N$31: track 9.40 -> 32.4 mm
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Other:
- board text added: "15v"
- board text added: "5v"
- board text added: "H1"
- board text added: "H2"
- board text added: "H3"
- board text added: "I"
- board text added: "March 2017"
- board text added: "SCL"
- board text added: "SDA"
- board text added: "Throttle"
- board text added: "Undervoltage"
- board text added: "V"
